Commit message: new

File: description/robot_core.xacro (robot description, xacro)
@@ -8,5 +8,5 @@
     <xacro:property name="wheel_radius" value="0.04"/>
     <xacro:property name="wheel_thickness" value="0.035"/>
-    <xacro:property name="wheel_mass" value="0.05"/>
+    <xacro:property name="wheel_mass" value="0.1"/>
     <xacro:property name="wheel_offset_x" value="0.115"/>
     <xacro:property name="wheel_offset_y" value="0.170"/>
@@ -37,5 +37,5 @@
     <link name="base_link"></link>
     <!-- BASE_FOOTPRINT LINK -->
-    <joint name="base_footprint_joint" type="fixed">
+    <!-- <joint name="base_footprint_joint" type="fixed">
         <parent link="base_link"/>
         <child link="base_footprint"/>
@@ -43,5 +43,5 @@
     </joint>
     <link name="base_footprint">
-    </link>
+    </link> -->
     <!-- CHASSIS LINK -->
     <joint name="chassis_joint" type="fixed">
