Commit message: changed laser_frame parent frame

File: description/lidar.xacro (robot description, xacro)
@@ -2,5 +2,5 @@
 <robot xmlns:xacro="http://www.ros.org/wiki/xacro" >
     <joint name="laser_joint" type="fixed">
-        <parent link="chassis"/>
+        <parent link="base_link"/>
         <child link="laser_frame"/>
         <origin xyz="0.1 0 0.450" rpy="0 0 0"/>

Commit message: changed laser_frame parent frame

File: description/lidar.xacro (robot description, xacro)
@@ -2,5 +2,5 @@
 <robot xmlns:xacro="http://www.ros.org/wiki/xacro" >
     <joint name="laser_joint" type="fixed">
-        <parent link="base_link"/>
+        <parent link="odom"/>
         <child link="laser_frame"/>
         <origin xyz="0.1 0 0.450" rpy="0 0 0"/>

Commit message: changed laser_frame parent frame

File: description/lidar.xacro (robot description, xacro)
@@ -2,5 +2,5 @@
 <robot xmlns:xacro="http://www.ros.org/wiki/xacro" >
     <joint name="laser_joint" type="fixed">
-        <parent link="odom"/>
+        <parent link="chassis"/>
         <child link="laser_frame"/>
         <origin xyz="0.1 0 0.450" rpy="0 0 0"/>
